File: eagle/T01_Synth_Glove_v4.sch (EAGLE design)
At the start: 72 parts, among them SW1 RESET_BUTTON, U1 ATMEGA328P, U2 ZLDO1117, U4 LT1013

Commit message: Schematic update, Started Prototype Board
Parts:
- removed TP15, TP20: PTR1B2,54, testpad:PTR1B2,54
- added C9: 100n, SparkFun-Capacitors:CAP0603-CAP
- added IC1: 317T, linear:317T
- added JP5, JP5*, JP6*, JP7*, JP8*, JP9*: 0, jumper:JP1E
- added R26: 100k, SparkFun-Resistors:RESISTOR0603
- R24: value NP -> 100k
Connections:
- removed net 5V: C2.1, JP2-2.1, JP2-2.2, R19.2, TP15.TP, U2.OUT@2, U2.OUT@4
- removed net 9V: JP2-1.1, JP2-1.2, U$7.1, U$8.+
- removed net V+: JP2*.1, U4.V+
- new net +9V: JP2*.1, JP2-1.1, JP2-1.2, U$7.1, U$8.+
- new net N$21: JP6*.1, R3.1
- new net N$25: JP7*.1, R2.1
- new net N$26: R26.2, U4.-INB
- new net N$27: JP8*.1, R18.1
- new net N$31: IC1.VO
- new net N$32: JP9*.1, R4.1
- new net N$35: R7.2, U4.OUTA
- new net N$36: U4.+INB
- new net N$39: C9.2, JP5.1
- new net N$40: IC1.VI, JP5.2, R24.1, U4.OUTB
- net +5V: now also C2.1, JP2-2.1, JP2-2.2, R19.2, U2.OUT@2, U2.OUT@4; no longer JP2*.2
- net GND: now also C9.1, R24.2, R26.1; no longer U4.+INB, U4.-INB, U4.OUTB
- net N$18: now also JP5*.1, R6.1; no longer JP4.1, R24.2, TP20.TP
- net N$2: now also JP5*.2, JP6*.2, JP7*.2, JP8*.2, JP9*.2; no longer R18.1, R2.1, R24.1, R3.1, R4.1, R6.1
- net N$34: now also JP2*.2, U4.V+; no longer R7.2, TP2.TP, U$1.SPKR+, U4.OUTA
- net PD6: no longer JP4.2
Other:
- note added: "Jumpers to allow for alternate tone generation scheme"
- note added: "Normal Operation mode"
- note added: "Programming mode"
- note added: "Summing and Amplification Stage"
- note removed: "Amplification Stage"
- moved on the sheet: JP1*, JP2*, JP2-1, JP2-2, JP4, PROG.JMP, R24, R7, R8, TP1, TP2
