File: eagle/T01_Synth_Glove_v5.brd (EAGLE design)
At the start: 63.5 x 38.1 mm, 79 parts, among them IC1 317T, SW1 RESET_BUTTON, U1 ATMEGA328P, U2 ZLDO1117, U4 LT1013

Commit message: issue 5 and greenberg requsts
Connections:
- net PB1 renamed B0
- net PC0 renamed A0
- net PC1 renamed A1
- net PC2 renamed A2
- net PC3 renamed D5
- net PC4 renamed D6
- net PC5 renamed D7
- net PD0 renamed D0
- net PD1 renamed D1
- net PD2 renamed D2
- net PD3 renamed D3
- net PD4 renamed D4
- net PD5 renamed B3
- net PD6 renamed B4
- removed net PB2: R3.2, TP14.TP, U1.14
- removed net PB3: PROG.JMP.3, R2.2, TP17.TP
- new net B1: R2.2, R3.2, TP14.TP, TP17.TP, U1.14
- new net B2: PROG.JMP.3
- net +5V: now also U1.6
- net N$31: now also U$1.1
Routing:
- net B4: track 31.4 -> 0.00 mm, vias 1 -> 0
- net +5V: track 97.3 -> 66.8 mm
- net B3: track 25.9 -> 0.00 mm
- net D4: track 17.7 -> 0.00 mm
- net PB2: track 17.4 -> 0.00 mm, vias 2 -> 0
- net B0: track 17.4 -> 0.00 mm, vias 2 -> 0
- net D3: track 15.0 -> 0.00 mm
- net A2: track 14.0 -> 0.00 mm
- net D7: track 13.8 -> 0.00 mm, vias 2 -> 0
- net A1: track 13.1 -> 0.00 mm
- net D2: track 12.5 -> 0.00 mm
- net D1: track 12.1 -> 0.00 mm
- net A0: track 12.0 -> 0.00 mm, vias 2 -> 0
- net PB3: track 11.5 -> 0.00 mm, vias 2 -> 0
- net D0: track 9.42 -> 0.00 mm, vias 2 -> 0
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