File: eagle/T01_Synth_Glove_v6.1.brd (EAGLE design)
At the start: 99.1 x 78.7 mm, 97 parts, among them SW1 RESET_BUTTON, U1 ATMEGA328P, U2 ZLDO1117, U3 LM386, U4 LT1013

Commit message: added mounting holes
Routing:
- net +9V: track 182.8 -> 180.4 mm
Changed lines of the file:
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@@
 <layer number="43" name="vRestrict" color="2" fill="10" visible="yes" active="yes"/>
 <layer number="44" name="Drills" color="7" fill="1" visible="no" active="yes"/>
-<layer number="45" name="Holes" color="7" fill="1" visible="no" active="yes"/>
+<layer number="45" name="Holes" color="7" fill="1" visible="yes" active="yes"/>
 <layer number="46" name="Milling" color="3" fill="1" visible="no" active="yes"/>
 <layer number="47" name="Measures" color="7" fill="1" visible="no" active="yes"/>
@@
 <text x="3.81" y="27.94" size="1.778" layer="104">GND </text>
 <text x="5.08" y="46.99" size="1.778" layer="104">9V</text>
+<hole x="4.318" y="4.318" drill="3.2"/>
+<hole x="94.742" y="74.422" drill="3.2"/>
 </plain>
 <attributes>
@@
 <wire x1="50.8" y1="76.2" x2="50.8" y2="73.66" width="1.778" layer="16"/>
 <wire x1="50.8" y1="73.66" x2="54.61" y2="73.66" width="1.778" layer="16"/>
-<wire x1="57.15" y1="73.66" x2="74.93" y2="73.66" width="1.778" layer="16"/>
-<wire x1="74.93" y1="73.66" x2="78.74" y2="77.47" width="1.778" layer="16"/>
-<wire x1="78.74" y1="77.47" x2="91.44" y2="77.47" width="1.778" layer="16"/>
-<wire x1="91.44" y1="77.47" x2="96.52" y2="72.39" width="1.778" layer="16"/>
-<wire x1="96.52" y1="72.39" x2="96.52" y2="59.69" width="1.778" layer="16"/>
+<wire x1="57.15" y1="73.66" x2="74.225009375" y2="72.108534375" width="1.778" layer="16"/>
+<wire x1="74.225009375" y1="72.108534375" x2="78.48620625" y2="75.9185375" width="1.778" layer="16"/>
+<wire x1="78.48620625" y1="75.9185375" x2="90.601484375" y2="75.6005625" width="1.778" layer="16"/>
+<wire x1="94.60243125" y1="69.371696875" x2="96.52" y2="59.69" width="1.778" layer="16"/>
 <wire x1="96.52" y1="59.69" x2="87.63" y2="59.69" width="1.778" layer="16"/>
 <wire x1="55.3212" y1="73.8378" x2="54.61" y2="73.66" width="0.254" layer="16"/>
@@
 <wire x1="56.4642" y1="73.8378" x2="54.61" y2="73.8378" width="0.3048" layer="16"/>
 <wire x1="54.61" y1="73.8378" x2="54.61" y2="73.66" width="0.3048" layer="16"/>
+<wire x1="94.60243125" y1="69.371696875" x2="90.470140625" y2="72.1113625" width="0.8128" layer="16"/>
+<wire x1="90.470140625" y1="72.1113625" x2="90.601484375" y2="75.6005625" width="0.8128" layer="16"/>
 </signal>
 <signal name="N$34">
