File: eagle/Old Revisions/T01_Synth_Glove_v3.1.brd (EAGLE design)
At the start: 63.5 x 38.1 mm, 72 parts, among them SW1 RESET_BUTTON, U1 ATMEGA328P, U2 ZLDO1117, U4 LT1013

Commit message: Schematic update, Started Prototype Board
Parts:
- removed JP4: 0, jumper:JP1
- removed R24: NP, SparkFun-Resistors:0603-RES
- removed TP20: PTR1B2,54, testpad:B2,54
- added JP5*, JP6*, JP7*, JP8*, JP9*: 0, jumper:JP1
Connections:
- removed net 5V: C2.1, JP2.3, JP2.4, R19.2, TP15.TP, U2.2, U2.4
- new net N$21: JP6*.1, R3.1
- new net N$25: JP7*.1, R2.1
- new net N$27: JP8*.1, R18.1
- new net N$32: JP9*.1, R4.1
- net +5V: now also C2.1, JP2.3, JP2.4, R19.2, TP15.TP, U2.2, U2.4
- net N$18: now also JP5*.1, R6.1; no longer JP4.1, R24.2, TP20.TP
- net N$2: now also JP5*.2, JP6*.2, JP7*.2, JP8*.2, JP9*.2; no longer R18.1, R2.1, R24.1, R3.1, R4.1, R6.1
- net PD6: no longer JP4.2
Routing:
- net 5V: track 37.6 -> 0.00 mm
- net N$2: track 20.0 -> 0.00 mm
- net N$18: track 16.6 -> 0.00 mm, vias 1 -> 0
- net PD6: track 38.0 -> 31.4 mm
Changed lines of the file:
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@@
 <?xml version="1.0" encoding="utf-8"?>
 <!DOCTYPE eagle SYSTEM "eagle.dtd">
-<eagle version="6.5.0">
+<eagle version="7.1.0">
 <drawing>
 <settings>
@@
 <pass name="Default">
 <param name="RoutingGrid" value="50mil"/>
+<param name="AutoGrid" value="1"/>
+<param name="Efforts" value="0"/>
+<param name="TopRouterVariant" value="1"/>
 <param name="tpViaShape" value="round"/>
 <param name="PrefDir.1" value="|"/>
@@
 <attribute name="NAME" x="21.594053125" y="2.68295" size="0.4064" layer="25" ratio="10" rot="R90"/>
 </element>
-<element name="JP4" library="jumper" package="JP1" value="0" x="46.63418125" y="14.99304375" smashed="yes">
-<attribute name="NAME" x="47.873065625" y="18.996759375" size="1.27" layer="25" ratio="10" rot="R180"/>
-</element>
 <element name="POT1" library="jumper" package="JP1" value="0" x="46.910565625" y="20.57216875" smashed="yes" rot="R90">
 <attribute name="NAME" x="43.674034375" y="20.485775" size="0.4064" layer="25" ratio="10" rot="R270"/>
@@
 <attribute name="NAME" x="23.110221875" y="11.38759375" size="0.4064" layer="25" font="vector"/>
 <attribute name="VALUE" x="22.983221875" y="9.48259375" size="0.4064" layer="27" font="vector"/>
-</element>
-<element name="R24" library="SparkFun-Resistors" package="0603-RES" value="NP" x="46.3721875" y="4.37033125" smashed="yes">
-<attribute name="NAME" x="45.4831875" y="5.13233125" size="0.4064" layer="25" font="vector"/>
-<attribute name="VALUE" x="44.1265625" y="3.44695" size="0.4064" layer="27" font="vector"/>
 </element>
 <element name="R25" library="SparkFun-Resistors" package="0603-RES" value="10k" x="33.234303125" y="30.131090625" smashed="yes" rot="R90">
@@
 <attribute name="NAME" x="57.17403125" y="6.6287875" size="0.6096" layer="25" ratio="10" rot="R90"/>
 </element>
-<element name="TP20" library="testpad" package="B2,54" value="PTR1B2,54" x="46.18626875" y="1.926671875" smashed="yes">
-<attribute name="TP_SIGNAL_NAME" value="" x="44.91626875" y="-1.248328125" size="1" layer="37"/>
-<attribute name="NAME" x="41.86826875" y="1.291671875" size="0.6096" layer="25" ratio="10"/>
-</element>
 <element name="TP3" library="testpad" package="B2,54" value="PTR1B2,54" x="23.36334375" y="26.405015625" smashed="yes" rot="R180">
 <attribute name="TP_SIGNAL_NAME" value="" x="24.63334375" y="29.580015625" size="1" layer="37" rot="R180"/>
@@
 <attribute name="VALUE" x="11.995390625" y="29.06438125" size="1.27" layer="27" ratio="10"/>
 </element>
+<element name="JP5*" library="jumper" package="JP1" value="0" x="-3.81" y="3.048"/>
+<element name="JP6*" library="jumper" package="JP1" value="0" x="-10.668" y="3.048"/>
+<element name="JP7*" library="jumper" package="JP1" value="0" x="-17.526" y="3.048"/>
+<element name="JP8*" library="jumper" package="JP1" value="0" x="-24.384" y="3.048"/>
+<element name="JP9*" library="jumper" package="JP1" value="0" x="-31.242" y="3.048"/>
 </elements>
 <signals>
@@
 <wire x1="18.542" y1="6.79334375" x2="18.579353125" y2="5.393790625" width="0.4064" layer="16"/>
 </signal>
-<signal name="5V">
-<contactref element="R19" pad="2"/>
-<contactref element="C2" pad="1"/>
-<contactref element="JP2" pad="4"/>
-<contactref element="JP2" pad="3"/>
-<contactref element="TP15" pad="TP"/>
-<contactref element="U2" pad="4"/>
-<contactref element="U2" pad="2"/>
-<wire x1="8.822678125" y1="7.856325" x2="8.55494375" y2="7.707140625" width="0.4064" layer="1"/>
-<wire x1="17.1596625" y1="20.925790625" x2="14.735059375" y2="17.463271875" width="1.016" layer="1"/>
-<wire x1="14.735059375" y1="17.463271875" x2="14.735059375" y2="14.732" width="1.016" layer="1"/>
-<wire x1="14.735059375" y1="14.732" x2="14.735059375" y2="11.265271875" width="1.016" layer="1"/>
-<wire x1="10.03605625" y1="14.7873625" x2="14.735059375" y2="14.732" width="1.016" layer="1"/>
-<wire x1="10.03605625" y1="14.7873625" x2="7.897075" y2="14.76785625" width="1.016" layer="1"/>
-<wire x1="7.897075" y1="14.76785625" x2="8.01770625" y2="9.19264375" width="1.016" layer="1"/>
-<wire x1="8.01770625" y1="9.19264375" x2="8.55494375" y2="7.707140625" width="1.016" layer="1"/>
-<wire x1="8.55494375" y1="5.167140625" x2="8.55494375" y2="7.707140625" width="1.016" layer="1"/>
-<wire x1="4.92294375" y1="15.169715625" x2="10.00294375" y2="17.463271875" width="1.016" layer="1"/>
-<wire x1="10.00294375" y1="17.463271875" x2="14.735059375" y2="17.463271875" width="1.016" layer="1"/>
-</signal>
 <signal name="N$6">
 <contactref element="U1" pad="7"/>
@@
 <contactref element="R4" pad="2"/>
 <contactref element="TP19" pad="TP"/>
-<contactref element="JP4" pad="2"/>
 <wire x1="27.5107" y1="15.158621875" x2="27.32184375" y2="13.21344375" width="0.4064" layer="1"/>
 <wire x1="27.32184375" y1="13.21344375" x2="29.446553125" y2="11.284725" width="0.4064" layer="1"/>
@@
 <wire x1="39.95069375" y1="6.17255" x2="41.9321125" y2="8.15396875" width="0.4064" layer="16"/>
 <wire x1="41.9321125" y1="8.15396875" x2="41.9321125" y2="11.560975" width="0.4064" layer="16"/>
-<wire x1="41.9321125" y1="11.560975" x2="46.63418125" y2="16.26304375" width="0.4064" layer="16"/>
 </signal>
 <signal name="PD7">
@@
 <wire x1="22.58260625" y1="19.86604375" x2="22.597428125" y2="19.851221875" width="0.6096" layer="1" curve="90"/>
 <wire x1="22.597428125" y1="19.851221875" x2="25.2181" y2="19.851221875" width="0.6096" layer="1"/>
+<contactref element="JP2" pad="4"/>
+<contactref element="C2" pad="1"/>
+<contactref element="U2" pad="2"/>
+<contactref element="JP2" pad="3"/>
+<contactref element="R19" pad="2"/>
+<contactref element="U2" pad="4"/>
+<contactref element="TP15" pad="TP"/>
+<wire x1="20.944540625" y1="19.833740625" x2="17.1596625" y2="20.925790625" width="0" layer="19" extent="1-1"/>
+<wire x1="14.735059375" y1="17.463271875" x2="17.1596625" y2="20.925790625" width="0" layer="19" extent="1-1"/>
+<wire x1="10.03605625" y1="14.7873625" x2="14.735059375" y2="17.463271875" width="0" layer="19" extent="1-1"/>
+<wire x1="4.92294375" y1="15.169715625" x2="10.03605625" y2="14.7873625" width="0" layer="19" extent="1-1"/>
+<wire x1="14.735059375" y1="11.265271875" x2="10.03605625" y2="14.7873625" width="0" layer="19" extent="1-1"/>
+<wire x1="8.55494375" y1="7.707140625" x2="14.735059375" y2="11.265271875" width="0" layer="19" extent="1-1"/>
+<wire x1="8.55494375" y1="5.167140625" x2="8.55494375" y2="7.707140625" width="0" layer="19" extent="1-1"/>
 </signal>
 <signal name="N$1">
@@
 <wire x1="42.199353125" y1="29.18913125" x2="37.427253125" y2="26.063721875" width="0.4064" layer="1"/>
 </signal>
-<signal name="N$18">
-<contactref element="R24" pad="2"/>
-<contactref element="JP4" pad="1"/>
-<contactref element="TP20" pad="TP"/>
-<wire x1="46.18626875" y1="1.926671875" x2="47.2221875" y2="4.37033125" width="0.4064" layer="1"/>
-<wire x1="46.63418125" y1="13.72304375" x2="43.926071875" y2="2.40446875" width="0.4064" layer="16"/>
-<via x="43.926071875" y="2.40446875" extent="1-16" drill="0.5"/>
-<wire x1="43.926071875" y1="2.40446875" x2="46.18626875" y2="1.926671875" width="0.4064" layer="1"/>
-</signal>
 <signal name="N$19">
 </signal>
@@
 <signal name="N$2">
 <contactref element="U4" pad="1"/>
-<contactref element="R2" pad="1"/>
-<contactref element="R18" pad="1"/>
-<contactref element="R3" pad="1"/>
-<contactref element="R6" pad="1"/>
-<contactref element="R4" pad="1"/>
 <contactref element="TP1" pad="TP"/>
-<contactref element="R24" pad="1"/>
-<wire x1="42.730065625" y1="12.272665625" x2="42.776334375" y2="9.767071875" width="0.4064" layer="1"/>
-<wire x1="42.776334375" y1="9.767071875" x2="42.744215625" y2="6.865759375" width="0.4064" layer="1"/>
-<wire x1="42.75399375" y1="3.970790625" x2="42.744215625" y2="6.865759375" width="0.4064" layer="1"/>
-<wire x1="42.75399375" y1="3.970790625" x2="40.877453125" y2="1.6937125" width="0.4064" layer="1"/>
-<wire x1="42.75399375" y1="3.970790625" x2="45.5221875" y2="4.37033125" width="0.4064" layer="1"/>
-<wire x1="45.9743625" y1="11.14080625" x2="42.730065625" y2="12.272665625" width="0.4064" layer="1"/>
-<wire x1="42.830990625" y1="14.785590625" x2="42.730065625" y2="12.272665625" width="0.4064" layer="1"/>
+<contactref element="JP5*" pad="2"/>
+<contactref element="JP6*" pad="2"/>
+<contactref element="JP7*" pad="2"/>
+<contactref element="JP8*" pad="2"/>
+<contactref element="JP9*" pad="2"/>
+<wire x1="42.830990625" y1="14.785590625" x2="45.9743625" y2="11.14080625" width="0" layer="19" extent="1-1"/>
+<wire x1="-3.81" y1="4.318" x2="42.830990625" y2="14.785590625" width="0" layer="19" extent="1-1"/>
+<wire x1="-10.668" y1="4.318" x2="-3.81" y2="4.318" width="0" layer="19" extent="1-1"/>
+<wire x1="-17.526" y1="4.318" x2="-10.668" y2="4.318" width="0" layer="19" extent="1-1"/>
+<wire x1="-24.384" y1="4.318" x2="-17.526" y2="4.318" width="0" layer="19" extent="1-1"/>
+<wire x1="-31.242" y1="4.318" x2="-24.384" y2="4.318" width="0" layer="19" extent="1-1"/>
 </signal>
 <signal name="N$28">
@@
 <signal name="N$33">
 </signal>
+<signal name="N$18">
+<contactref element="R6" pad="1"/>
+<contactref element="JP5*" pad="1"/>
+<wire x1="-3.81" y1="1.778" x2="42.744215625" y2="6.865759375" width="0" layer="19" extent="1-1"/>
+</signal>
+<signal name="N$21">
+<contactref element="R3" pad="1"/>
+<contactref element="JP6*" pad="1"/>
+<wire x1="-10.668" y1="1.778" x2="42.776334375" y2="9.767071875" width="0" layer="19" extent="1-1"/>
+</signal>
+<signal name="N$25">
+<contactref element="R2" pad="1"/>
+<contactref element="JP7*" pad="1"/>
+<wire x1="-17.526" y1="1.778" x2="42.730065625" y2="12.272665625" width="0" layer="19" extent="1-1"/>
+</signal>
+<signal name="N$27">
+<contactref element="R18" pad="1"/>
+<contactref element="JP8*" pad="1"/>
+<wire x1="-24.384" y1="1.778" x2="40.877453125" y2="1.6937125" width="0" layer="19" extent="1-1"/>
+</signal>
+<signal name="N$32">
+<contactref element="R4" pad="1"/>
+<contactref element="JP9*" pad="1"/>
+<wire x1="-31.242" y1="1.778" x2="42.75399375" y2="3.970790625" width="0" layer="19" extent="1-1"/>
+</signal>
 </signals>
