File: eagle/Prototype Board/T01_Synth_Glove_Prototype_Board.brd (EAGLE design)
At the start: 76.2 x 76.2 mm, 61 parts, among them SW1 RESET_BUTTON, U1 ATMEGA328P, U2 ZLDO1117

Commit message: Update, more CAM files
Parts:
- removed PROTOJMP2, PROTOJMP3, PROTOJMP4: PTR1B2,54, testpad:B2,54
- added PROG_5V, PROG_RESET, PROG_SCK: PTR1B2,54, testpad:B2,54
- moved PROTOJMP1 16.2 mm to (44.6, 19.4)
- moved TP7 10.3 mm to (20.8, 35.5)
- moved PROTOJMP5 10.0 mm to (6.38, 28.1)
- moved TP6 9.84 mm to (23.8, 36.5)
- moved JP3 9.62 mm to (3.00, 28.9)
- moved TP5 9.35 mm to (27.4, 35.5)
- moved R13 9.06 mm to (25.2, 40.0)
- moved R14 9.06 mm to (22.6, 40.0)
- moved TP4 8.71 mm to (30.6, 36.8)
- moved R12 8.40 mm to (28.2, 39.8)
- moved R11 8.35 mm to (30.8, 39.9)
- moved POT1 8.25 mm to (57.8, 22.9)
- moved C8 8.20 mm to (49.7, 18.4)
- moved C3 8.20 mm to (24.5, 27.4)
- moved C1 8.20 mm to (14.6, 21.8)
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Connections:
- new net JP3: PROG_SCK.TP, SV1.3
- new net N$2: PROG_5V.TP, SV1.5
- new net PJ4: PROG_RESET.TP, SV1.6
- net +5V: no longer PROTOJMP2.TP, SV1.5
- net RESET: no longer PROTOJMP3.TP, SV1.3
- net SCK: no longer PROTOJMP4.TP, SV1.6
Routing:
- net +5V: track 182.0 -> 195.3 mm
- net PC3: track 16.8 -> 21.3 mm
- net PJ4: track 0.00 -> 3.66 mm
- net N$2: track 0.00 -> 3.44 mm
- net SCK: track 7.41 -> 4.00 mm
- net JP3: track 0.00 -> 3.26 mm
- net RESET: track 20.4 -> 17.2 mm
- net PC4: track 14.8 -> 17.3 mm
- net +9V: track 7.60 -> 10.1 mm
- net PD4: track 18.3 -> 20.7 mm
- net PC5: track 12.6 -> 14.4 mm
- net PC2: track 16.2 -> 18.0 mm
- net PD3: track 15.9 -> 17.6 mm
- net N$15: track 17.2 -> 15.7 mm
- net N$13: track 17.2 -> 15.7 mm
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Other:
- board size 76.2 x 76.2 mm -> 68.6 x 50.8 mm

Commit message: Revisions and more CAM
Parts:
- removed JP1: 0, jumper:JP8Q
- removed R15, R16, R17: 1k, SparkFun-Resistors:0603-RES
- removed TP10, TP8, TP9: PTR1B2,54, testpad:B2,54
- added C12, C13, C14, C15, C16: 100n, SparkFun-Capacitors:0603-CAP
- added R3, R4, R6, R7, R8: 1k, SparkFun-Resistors:0603-RES
- added SW2, SW5, SW6, SW8, SW9: RESET_BUTTON, Synth_Glove:RESET_BUTTON
- moved R10 7.16 mm to (33.0, 46.6)
- moved R12 6.76 mm to (27.7, 46.6)
- moved R11 6.75 mm to (30.3, 46.6)
- moved R14 6.73 mm to (21.7, 46.6)
- moved R13 6.67 mm to (24.8, 46.6)
- moved SW1 2.54 mm to (38.7, 41.5)
- moved PROTOJMP6 1.94 mm to (37.7, 35.1)
Connections:
- removed net N$23: JP1.11, R17.2
- removed net N$3: JP1.9, R10.2
- removed net N$4: JP1.7, R11.2
- net +5V: now also R3.1, R4.2, R6.2, R7.2, R8.2; no longer JP1.10, JP1.12, JP1.14, JP1.16, JP1.2, JP1.4, JP1.6, JP1.8
- net GND: now also C12.1, C13.1, C14.1, C15.1, C16.1, SW2.3, SW2.4, SW5.3, SW5.4, SW6.3, SW6.4, SW8.3, SW8.4, SW9.3, SW9.4
- net N$11: now also R7.1, SW6.1, SW6.2; no longer JP1.3
- net N$12: now also R12.2, R6.1, SW5.1, SW5.2; no longer JP1.1, R14.2
- net N$13: now also R11.2, R4.1, SW9.1, SW9.2; no longer JP1.15, R15.2
- net N$15: now also R10.2, R3.2, SW2.1, SW2.2; no longer JP1.13, R16.2
- net N$5: now also R14.2, R8.1, SW8.1, SW8.2; no longer JP1.5, R12.2
- net PC3: no longer R15.1, TP8.TP
- net PC4: no longer R16.1, TP9.TP
- net PC5: no longer R17.1, TP10.TP
- net PD0: now also C16.2
- net PD1: now also C15.2
- net PD2: now also C14.2
- net PD3: now also C13.2
- net PD4: now also C12.2
Routing:
- net +5V: track 195.3 -> 273.5 mm
- net N$5: track 4.77 -> 22.1 mm
- net N$23: track 16.8 -> 0.00 mm
- net N$11: track 4.72 -> 19.9 mm
- net N$12: track 4.72 -> 15.8 mm
- net PC3: track 21.3 -> 12.0 mm
- net PC5: track 14.4 -> 5.61 mm
- net PC4: track 17.3 -> 9.77 mm
- net PD0: track 11.0 -> 18.2 mm
- net N$15: track 15.7 -> 22.7 mm
- net PD1: track 13.2 -> 20.2 mm
- net PD3: track 17.6 -> 24.6 mm
- net PD2: track 15.0 -> 21.5 mm
- net PD4: track 20.7 -> 27.2 mm
- net N$3: track 5.12 -> 0.00 mm
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Other:
- board size 68.6 x 50.8 mm -> 68.6 x 71.1 mm
