File: eagle/Prototype Board/T01_Synth_Glove_Prototype_Board.sch (EAGLE design)
At the start: 61 parts, among them SW1 RESET_BUTTON, U1 ATMEGA328P, U2 ZLDO1117

Commit message: test board revisions
Connections:
- net N$22: no longer PROTOJMP6.TP
- net RESET: now also PROTOJMP6.TP
Other:
- moved on the sheet: R1
Changed lines of the file:
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@@
 <instances>
 <instance part="U1" gate="G$1" x="88.9" y="-12.7"/>
-<instance part="R1" gate="G$1" x="63.5" y="19.05" rot="R90"/>
+<instance part="R1" gate="G$1" x="58.42" y="19.05" rot="R90"/>
 <instance part="C1" gate="G$1" x="11.43" y="77.47"/>
 <instance part="GND1" gate="1" x="58.42" y="-45.72"/>
@@
 <pinref part="U1" gate="G$1" pin="PC6(/RESET)"/>
 <pinref part="R1" gate="G$1" pin="1"/>
-<wire x1="66.04" y1="12.7" x2="63.5" y2="13.97" width="0.1524" layer="91"/>
+<wire x1="66.04" y1="12.7" x2="58.42" y2="13.97" width="0.1524" layer="91"/>
 <wire x1="66.04" y1="12.7" x2="53.34" y2="12.7" width="0.1524" layer="91"/>
 <junction x="66.04" y="12.7"/>
@@
 <wire x1="53.34" y1="12.7" x2="53.34" y2="19.05" width="0.1524" layer="91"/>
 <pinref part="R25" gate="G$1" pin="1"/>
+<pinref part="PROTOJMP6" gate="G$1" pin="TP"/>
+<wire x1="73.66" y1="25.4" x2="66.04" y2="25.4" width="0.1524" layer="91"/>
+<wire x1="66.04" y1="25.4" x2="66.04" y2="12.7" width="0.1524" layer="91"/>
 </segment>
 </net>
@@
 <wire x1="63.5" y1="33.02" x2="63.5" y2="30.48" width="0.1524" layer="91"/>
 <pinref part="R1" gate="G$1" pin="2"/>
-<wire x1="63.5" y1="24.13" x2="63.5" y2="25.4" width="0.1524" layer="91"/>
 <junction x="63.5" y="30.48"/>
-<pinref part="PROTOJMP6" gate="G$1" pin="TP"/>
-<wire x1="63.5" y1="25.4" x2="63.5" y2="30.48" width="0.1524" layer="91"/>
-<wire x1="73.66" y1="25.4" x2="63.5" y2="25.4" width="0.1524" layer="91"/>
-<junction x="63.5" y="25.4"/>
-</segment>
-</net>
+<wire x1="58.42" y1="24.13" x2="63.5" y2="30.48" width="0.1524" layer="91"/>
+</segment>
+</net>

Commit message: Update, more CAM files
Parts:
- renumbered PROTOJMP2 to PROG_5V, PROTOJMP3 to PROG_SCK, PROTOJMP4 to PROG_RESET
Connections:
- new net JP3: PROG_SCK.TP, SV1.3
- new net N$2: PROG_5V.TP, SV1.5
- new net PJ4: PROG_RESET.TP, SV1.6
- net +5V: no longer PROG_5V.TP, SV1.5
- net RESET: no longer PROG_SCK.TP, SV1.3
- net SCK: no longer PROG_RESET.TP, SV1.6
Changed lines of the file:
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@@
 <part name="5V7" library="supply2" deviceset="+5V" device=""/>
 <part name="5V8" library="supply2" deviceset="+5V" device=""/>
-<part name="5V4" library="supply2" deviceset="+5V" device=""/>
 <part name="5V9" library="supply2" deviceset="+5V" device=""/>
 <part name="SUPPLY1" library="supply2" deviceset="+9V" device=""/>
 <part name="PROTOJMP1" library="testpad" deviceset="PTR1" device="B2,54"/>
-<part name="PROTOJMP2" library="testpad" deviceset="PTR1" device="B2,54"/>
-<part name="PROTOJMP3" library="testpad" deviceset="PTR1" device="B2,54"/>
-<part name="PROTOJMP4" library="testpad" deviceset="PTR1" device="B2,54"/>
+<part name="PROG_5V" library="testpad" deviceset="PTR1" device="B2,54"/>
+<part name="PROG_SCK" library="testpad" deviceset="PTR1" device="B2,54"/>
+<part name="PROG_RESET" library="testpad" deviceset="PTR1" device="B2,54"/>
 <part name="PROTOJMP5" library="testpad" deviceset="PTR1" device="B2,54"/>
 <part name="PROTOJMP6" library="testpad" deviceset="PTR1" device="B2,54"/>
@@
 <attribute name="VALUE" x="40.259" y="1.143" size="1.778" layer="96"/>
 </instance>
-<instance part="5V4" gate="+5V" x="190.5" y="-36.83"/>
 <instance part="5V9" gate="+5V" x="53.34" y="99.06"/>
 <instance part="SUPPLY1" gate="G$1" x="-22.86" y="99.06"/>
 <instance part="PROTOJMP1" gate="G$1" x="110.49" y="-53.34" rot="R270"/>
-<instance part="PROTOJMP2" gate="G$1" x="200.66" y="-40.64" rot="R90"/>
-<instance part="PROTOJMP3" gate="G$1" x="200.66" y="-46.99" rot="R90"/>
-<instance part="PROTOJMP4" gate="G$1" x="162.56" y="-38.1" rot="R270"/>
+<instance part="PROG_5V" gate="G$1" x="200.66" y="-40.64" rot="R90"/>
+<instance part="PROG_SCK" gate="G$1" x="200.66" y="-46.99" rot="R90"/>
+<instance part="PROG_RESET" gate="G$1" x="162.56" y="-38.1" rot="R270"/>
 <instance part="PROTOJMP5" gate="G$1" x="60.96" y="96.52" rot="R90"/>
 <instance part="PROTOJMP6" gate="G$1" x="76.2" y="25.4" rot="R90"/>
@@
 <junction x="116.84" y="-45.72"/>
 </segment>
-<segment>
-<pinref part="SV1" gate="1" pin="6"/>
-<wire x1="167.64" y1="-44.45" x2="165.1" y2="-44.45" width="0.1524" layer="91"/>
-<wire x1="165.1" y1="-44.45" x2="165.1" y2="-40.64" width="0.1524" layer="91"/>
-<wire x1="165.1" y1="-40.64" x2="157.48" y2="-40.64" width="0.1524" layer="91"/>
-<label x="157.48" y="-40.64" size="1.778" layer="95" rot="R180" xref="yes"/>
-<pinref part="PROTOJMP4" gate="G$1" pin="TP"/>
-<wire x1="165.1" y1="-40.64" x2="165.1" y2="-38.1" width="0.1524" layer="91"/>
-<junction x="165.1" y="-40.64"/>
-</segment>
 </net>
 <net name="RESET" class="0">
-<segment>
-<label x="194.31" y="-54.61" size="1.778" layer="95" xref="yes"/>
-<wire x1="187.96" y1="-54.61" x2="194.31" y2="-54.61" width="0.1524" layer="91"/>
-<pinref part="PROTOJMP3" gate="G$1" pin="TP"/>
-<pinref part="SV1" gate="1" pin="3"/>
-<wire x1="198.12" y1="-46.99" x2="187.96" y2="-46.99" width="0.1524" layer="91"/>
-<wire x1="187.96" y1="-46.99" x2="182.88" y2="-46.99" width="0.1524" layer="91"/>
-<wire x1="187.96" y1="-54.61" x2="187.96" y2="-46.99" width="0.1524" layer="91"/>
-<junction x="187.96" y="-46.99"/>
-</segment>
 <segment>
 <pinref part="U1" gate="G$1" pin="PC6(/RESET)"/>
@@
 </segment>
 <segment>
-<pinref part="SV1" gate="1" pin="5"/>
-<wire x1="182.88" y1="-44.45" x2="182.88" y2="-40.64" width="0.1524" layer="91"/>
-<wire x1="182.88" y1="-40.64" x2="190.5" y2="-40.64" width="0.1524" layer="91"/>
-<wire x1="190.5" y1="-40.64" x2="190.5" y2="-39.37" width="0.1524" layer="91"/>
-<pinref part="5V4" gate="+5V" pin="+5V"/>
-<pinref part="PROTOJMP2" gate="G$1" pin="TP"/>
-<wire x1="190.5" y1="-40.64" x2="198.12" y2="-40.64" width="0.1524" layer="91"/>
-<junction x="190.5" y="-40.64"/>
-</segment>
-<segment>
 <wire x1="53.34" y1="86.36" x2="45.72" y2="86.36" width="0.1524" layer="91"/>
 <wire x1="53.34" y1="83.82" x2="53.34" y2="86.36" width="0.1524" layer="91"/>
@@
 </segment>
 </net>
+<net name="PJ4" class="0">
+<segment>
+<pinref part="SV1" gate="1" pin="6"/>
+<wire x1="167.64" y1="-44.45" x2="165.1" y2="-44.45" width="0.1524" layer="91"/>
+<wire x1="165.1" y1="-44.45" x2="165.1" y2="-38.1" width="0.1524" layer="91"/>
+<pinref part="PROG_RESET" gate="G$1" pin="TP"/>
+</segment>
+</net>
+<net name="JP3" class="0">
+<segment>
+<pinref part="PROG_SCK" gate="G$1" pin="TP"/>
+<pinref part="SV1" gate="1" pin="3"/>
+<wire x1="198.12" y1="-46.99" x2="182.88" y2="-46.99" width="0.1524" layer="91"/>
+</segment>
+</net>
+<net name="N$2" class="0">
+<segment>
+<pinref part="SV1" gate="1" pin="5"/>
+<wire x1="182.88" y1="-44.45" x2="182.88" y2="-40.64" width="0.1524" layer="91"/>
+<pinref part="PROG_5V" gate="G$1" pin="TP"/>
+<wire x1="182.88" y1="-40.64" x2="198.12" y2="-40.64" width="0.1524" layer="91"/>
+</segment>
+</net>

Commit message: Revisions and more CAM
Parts:
- removed JP1: 0, jumper:JP8QE
- removed R15, R16, R17: 1k, SparkFun-Resistors:RESISTOR0603
- removed TP10, TP8, TP9: PTR1B2,54, testpad:PTR1B2,54
- added C12, C13, C14, C15, C16: 100n, SparkFun-Capacitors:CAP0603-CAP
- added R3, R4, R6, R7, R8: 1k, SparkFun-Resistors:RESISTOR0603
- added SW2, SW5, SW6, SW8, SW9: RESET_BUTTON, Synth_Glove:RESET_BUTTON
Connections:
- removed net N$23: JP1-6.1, R17.2
- removed net N$3: JP1-5.1, R10.2
- removed net N$4: JP1-4.1, R11.2
- net +5V: now also R3.1, R4.2, R6.2, R7.2, R8.2; no longer JP1-1.2, JP1-2.2, JP1-3.2, JP1-4.2, JP1-5.2, JP1-6.2, JP1-7.2, JP1-8.2
- net GND: now also C12.1, C13.1, C14.1, C15.1, C16.1, SW2.3, SW2.4, SW5.3, SW5.4, SW6.3, SW6.4, SW8.3, SW8.4, SW9.3, SW9.4
- net N$11: now also R7.1, SW6.1, SW6.2; no longer JP1-2.1
- net N$12: now also R12.2, R6.1, SW5.1, SW5.2; no longer JP1-1.1, R14.2
- net N$13: now also R11.2, R4.1, SW9.1, SW9.2; no longer JP1-8.1, R15.2
- net N$15: now also R10.2, R3.2, SW2.1, SW2.2; no longer JP1-7.1, R16.2
- net N$5: now also R14.2, R8.1, SW8.1, SW8.2; no longer JP1-3.1, R12.2
- net PC3: no longer R15.1, TP8.TP
- net PC4: no longer R16.1, TP9.TP
- net PC5: no longer R17.1, TP10.TP
- net PD0: now also C16.2
- net PD1: now also C15.2
- net PD2: now also C14.2
- net PD3: now also C13.2
- net PD4: now also C12.2
Other:
- moved on the sheet: R10, R11, R12, R13, R14, TP3, TP4, TP5, TP6, TP7
